Commit message: fixed pose, sensors, and improved code

File: urdf/auv/auv.urdf.xacro (robot description, xacro)
@@ -4,11 +4,9 @@
   <xacro:include filename="$(find auv_description)/urdf/sensors/imu.urdf.xacro"/>
   <xacro:include filename="$(find auv_description)/urdf/sensors/magnetometer.urdf.xacro"/>
-  <!-- <xacro:include filename="$(find auv_description)/urdf/sensors/camera.urdf.xacro"/> -->
   <xacro:include filename="$(find auv_description)/urdf/thrusters/thrusters.urdf.xacro"/>
   <link name="base_link">
-    <!-- Inertial -->
     <inertial>
       <origin xyz="0 0 -0.59" rpy="0 0 0"/>
-      <mass value="1862.87"/>
+      <mass value="2464.1"/>
       <inertia
         ixx="525.39"
@@ -19,5 +17,4 @@
         izz="691.23"/>
     </inertial>
-    <!-- Visual mesh -->
     <visual>
       <origin xyz="0 0 0" rpy="0 0 0"/>
@@ -26,5 +23,4 @@
       </geometry>
     </visual>
-    <!-- Bottom plate -->
     <collision>
       <origin xyz="0 0 -0.75" rpy="0 0 0"/>
@@ -33,5 +29,4 @@
       </geometry>
     </collision>
-    <!-- Top plate -->
     <collision>
       <origin xyz="0 0 0.60" rpy="0 0 0"/>
@@ -40,5 +35,4 @@
       </geometry>
     </collision>
-    <!-- Left side -->
     <collision>
       <origin xyz="-0.20 0.70 -0.15" rpy="0 0 0"/>
@@ -47,5 +41,4 @@
       </geometry>
     </collision>
-    <!-- Right side -->
     <collision>
       <origin xyz="0.20 -0.70 -0.15" rpy="0 0 0"/>
@@ -54,16 +47,11 @@
       </geometry>
     </collision>
-  </link>
     <gazebo>
       <plugin
         filename="gz-sim-hydrodynamics-system"
         name="gz::sim::systems::Hydrodynamics">
-        <!-- Ocean physics options -->
         <disable_coriolis>false</disable_coriolis>
         <disable_added_mass>false</disable_added_mass>
         <water_density>1028</water_density>
-        <!-- Target link -->
-        <link_name>base_link</link_name>
-        <!-- Added mass -->
         <xDotU>-4.876161</xDotU>
         <yDotV>-126.324739</yDotV>
@@ -72,5 +60,4 @@
         <mDotQ>-33.46</mDotQ>
         <nDotR>-33.46</nDotR>
-        <!-- Linear Drag Coefficients -->
         <xU>-74.82</xU>
         <yV>-69.48</yV>
@@ -79,5 +66,4 @@
         <mQ>-309.77</mQ>
         <nR>-105</nR>
-        <!-- Quadratic Drag Coefficients -->
         <xUabsU>-748.22</xUabsU>
         <yVabsV>-992.53</yVabsV>
@@ -87,4 +73,7 @@
         <nRabsR>-523.27</nRabsR>
       </plugin>
+    </gazebo>
+  </link>
+  <gazebo>
       <plugin
         filename="gz-sim-odometry-publisher-system"
@@ -95,4 +84,4 @@
         <odom_publish_frequency>100</odom_publish_frequency>
       </plugin>
-    </gazebo>
+  </gazebo>
 </robot>

File: urdf/sensors/camera.urdf.xacro (robot description, xacro)
@@ -51,8 +51,8 @@
       </camera>
       <always_on>1</always_on>
-      <topic>/auv/camera/image_raw</topic>
+      <topic>/auv/camera/image</topic>
       <update_rate>30</update_rate>
       <visualize>true</visualize>
     </sensor>
-    </sensor>
 </gazebo>
+</robot>

File: urdf/thrusters/thrusters.urdf.xacro (robot description, xacro)
@@ -1,6 +1,4 @@
 <?xml version="1.0" ?>
 <robot xmlns:xacro="http://www.ros.org/wiki/xacro">
-<?xml version="1.0"?>
-<robot xmlns:xacro="http://ros.org/wiki/xacro" name="rexrov_thrusters">
   <!-- Thruster macro -->
   <xacro:macro name="thruster" params="name xyz rpy">
